File: layout/P1/layou1/layou1.sch (KiCad schematic (older format))
At the start: 1 part

Commit message: b
Parts:
- added U1: MDBT42QA, mFootprintLib:MDBT42Q, symbol mSymbolLib:MDBT42QA
- added U2: BT407, mFootprintLib:BT407, symbol mSymbolLib:BT407
- gave numbers to parts that had none: 1
Changed lines of the file:
@@
 EESchema Schematic File Version 4
+LIBS:layou1-cache
 EELAYER 30 0
 EELAYER END
@@
 $EndDescr
 $Comp
-L Connector:4P2C_Shielded J?
+L Connector:4P2C_Shielded J1
 U 1 1 5E450A27
 P 5600 3750
-F 0 "J?" H 5657 4217 50  0000 C CNN
+F 0 "J1" H 5657 4217 50  0000 C CNN
 F 1 "4P2C_Shielded" H 5657 4126 50  0000 C CNN
 F 2 "" V 5600 3800 50  0001 C CNN
@@
 	1    0    0    -1
 $EndComp
+$Comp
+L mSymbolLib:BT407 U2
+U 1 1 5E451B18
+P 3700 4300
+F 0 "U2" H 3708 4686 59  0000 C CNN
+F 1 "BT407" H 3708 4581 59  0000 C CNN
+F 2 "mFootprintLib:BT407" H 3650 4000 50  0001 C CNN
+F 3 "" H 3700 4300 50  0001 C CNN
+	1    3700 4300
+	1    0    0    -1
+$EndComp
+$Comp
+L mSymbolLib:MDBT42QA U1
+U 1 1 5E452394
+P 1350 3150
+F 0 "U1" H 2050 5536 59  0000 C CNN
+F 1 "MDBT42QA" H 2050 5431 59  0000 C CNN
+F 2 "mFootprintLib:MDBT42Q" H 1350 3150 50  0001 C CNN
+F 3 "" H 1350 3150 50  0001 C CNN
+	1    1350 3150
+	1    0    0    -1
+$EndComp
